File: springreverb_lm386_2.kicad_sch (KiCad schematic)
At the start: 64 parts, among them J1 IN, J10 FromSW, J11 To_Tank, J12 From_Tank, J13 FromGND, J14 From, J15 VR_3_1, J16 VR4_1, J17 OUT, J2 Vin, J3 GND, J4 VR1_3, J5 toC6, J6 toC7, J7 VR2_3, J8 VR_2_2, J9 To, SW1 SW_SPDT, SW2 SW_SPST, U1 TL072, U2 TC1044S, U3 LM386

Commit message: 不要なものを削除した
Parts:
- removed C10, C8: 10u, Capacitor_THT:CP_Radial_D5.0mm_P2.50mm, symbol Device:C_Small_US
- removed C12, C2: 1000u, Capacitor_THT:CP_Radial_D13.0mm_P5.00mm, symbol Device:C_Small_US
- removed C13, C4: 0.1u, Capacitor_THT:C_Rect_L4.0mm_W2.5mm_P2.50mm, symbol Device:C_Small
- removed C16, C19: 100u, Capacitor_THT:CP_Radial_D7.5mm_P2.50mm, symbol Device:C_Small_US
- removed C21: 0.047uF, symbol Device:C_Small
- removed C5: 4700p, MyLibrary:9.3_4.3_p7.5, symbol Device:C_Small
- removed J10: FromSW, MyLibrary:PinHeader_1x01_P2.54mm_Vertical, symbol Connector:Conn_01x01_Pin
- removed J15: VR_3_1, MyLibrary:PinHeader_1x01_P2.54mm_Vertical, symbol Connector:Conn_01x01_Pin
- removed J5: toC6, MyLibrary:PinHeader_1x01_P2.54mm_Vertical, symbol Connector:Conn_01x01_Pin
- removed J6: toC7, MyLibrary:PinHeader_1x01_P2.54mm_Vertical, symbol Connector:Conn_01x01_Pin
- removed R3, R6: 10, Resistor_THT:R_Axial_DIN0204_L3.6mm_D1.6mm_P7.62mm_Horizontal, symbol Device:R_Small
- removed R7, R9: 470, Resistor_THT:R_Axial_DIN0204_L3.6mm_D1.6mm_P7.62mm_Horizontal, symbol Device:R_Small
- removed SW1: SW_SPDT, symbol Switch:SW_SPDT
- removed SW2: SW_SPST, symbol Switch:SW_SPST
- removed U2: TC1044S, MyLibrary:CERDIP-8_W7.62mm_SideBrazed_Socket, symbol MyLibrary:TC1044S
- removed VR1, VR3: B20k, symbol Device:R_Potentiometer
- J2: value Vin -> 15V
- J3: value GND -> 0V
- J4: value VR1_3 -> 15V
Connections:
- net at C7.1, U3.6 (V+): no longer J2.1 (Pin_1)
- net at C3.2: now also R4.2; no longer J4.1 (Pin_1)
- net at R5.2: now also C6.2, R4.1; no longer R4.2
- net GND renamed GND1
- net GND1: no longer C11.2, C7.2, J3.1 (Pin_1), U3.2 (-), U3.4 (GND)
- new net GND2: C11.2, C7.2, U3.2 (-), U3.4 (GND)
Other:
- moved on the sheet: C6, J2, J3, R4, R5

Commit message: 一旦配置完了
Parts:
- removed J3: 0V, MyLibrary:PinHeader_1x01_P2.54mm_Vertical, symbol Connector:Conn_01x01_Pin
- added J15: VR4_3, MyLibrary:PinHeader_1x01_P2.54mm_Vertical, symbol Connector:Conn_01x01_Pin
- added J16: OUT_GND, MyLibrary:PinHeader_1x01_P2.54mm_Vertical, symbol Connector:Conn_01x01_Pin
- added J2: IN_GND, MyLibrary:PinHeader_1x01_P2.54mm_Vertical, symbol Connector:Conn_01x01_Pin
- added J5: GND2, MyLibrary:PinHeader_1x01_P2.54mm_Vertical, symbol Connector:Conn_01x01_Pin
- added J6: +15v2, MyLibrary:PinHeader_1x01_P2.54mm_Vertical, symbol Connector:Conn_01x01_Pin
- C4: renamed from C17; footprint Capacitor_THT:C_Rect_L4.0mm_W2.5mm_P2.50mm -> Capacitor_THT:C_Disc_D5.0mm_W2.5mm_P2.50mm
- C5: renamed from C18; footprint Capacitor_THT:C_Rect_L4.0mm_W2.5mm_P2.50mm -> Capacitor_THT:C_Disc_D5.0mm_W2.5mm_P5.00mm
- J3: renamed from J2; value 15V -> +15v
- J4: value 15V -> -15v
- R3: renamed from R4; footprint (none) -> Resistor_THT:R_Axial_DIN0204_L3.6mm_D1.6mm_P7.62mm_Horizontal
- R4: renamed from R5; footprint (none) -> Resistor_THT:R_Axial_DIN0204_L3.6mm_D1.6mm_P7.62mm_Horizontal
- renumbered C15 to C10, C20 to C11, C22 to C12, C3 to C2, C6 to C3, C9 to C6, C11 to C8, C14 to C9, J11 to J10, J12 to J11, J13 to J12, J14 to J13, J16 to J14, R8 to R5, R10 to R6, R11 to R7, R12 to R8, U3 to U2, VR2 to VR1, VR4 to VR2
Connections:
- net GND1: now also J16.1 (Pin_1), J2.1 (Pin_1); no longer R5.2
- net GND2: now also R5.2, J5.1 (Pin_1)
- net at C5.1, U1.4 (V-): now also J4.1 (Pin_1)
- net at C4.1, U1.8 (V+): now also J3.1 (Pin_1)
- net at C7.1, U2.6 (V+): now also J6.1 (Pin_1)
- net at C11.2, VR2.3: now also J15.1 (Pin_1)
Other:
- moved on the sheet: C4, C5, J3, J4, U1C
